File: Chessboard-Hardware.kicad_sch (KiCad schematic)
At the start: 19 parts, among them IC1 SS49E, IC10 SS49E, IC11 SS49E, IC12 SS49E, IC13 SS49E, IC14 SS49E, IC15 SS49E, IC16 SS49E, IC2 SS49E, IC3 SS49E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

Commit message: PCB done
Parts:
- IC1, IC10, IC11, IC12, IC13, IC14, IC15, IC16, IC2, IC3, IC4, IC5, IC6, IC7, IC8, IC9: footprint TO130P160X410X300-3P -> Custom SamacSys Footprints:TO130P160X410X300-3P
Changed lines of the file:
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@@
 			)
 		)
-		(property "Footprint" "TO130P160X410X300-3P"
+		(property "Footprint" "Custom SamacSys Footprints:TO130P160X410X300-3P"
 			(at 110.82 119.38 0)
 			(effects
@@
 			)
 		)
-		(property "Footprint" "TO130P160X410X300-3P"
+		(property "Footprint" "Custom SamacSys Footprints:TO130P160X410X300-3P"
 			(at 257.48 33.02 0)
 			(effects
@@
 			)
 		)
-		(property "Footprint" "TO130P160X410X300-3P"
+		(property "Footprint" "Custom SamacSys Footprints:TO130P160X410X300-3P"
 			(at 72.72 119.38 0)
 			(effects
@@
 			)
 		)
-		(property "Footprint" "TO130P160X410X300-3P"
+		(property "Footprint" "Custom SamacSys Footprints:TO130P160X410X300-3P"
 			(at 148.92 119.38 0)
 			(effects
@@
 			)
 		)
-		(property "Footprint" "TO130P160X410X300-3P"
+		(property "Footprint" "Custom SamacSys Footprints:TO130P160X410X300-3P"
 			(at 53.67 119.38 0)
 			(effects
@@
 			)
 		)
-		(property "Footprint" "TO130P160X410X300-3P"
+		(property "Footprint" "Custom SamacSys Footprints:TO130P160X410X300-3P"
 			(at 314.63 33.02 0)
 			(effects
@@
 			)
 		)
-		(property "Footprint" "TO130P160X410X300-3P"
+		(property "Footprint" "Custom SamacSys Footprints:TO130P160X410X300-3P"
 			(at 295.58 33.02 0)
 			(effects
@@
 			)
 		)
-		(property "Footprint" "TO130P160X410X300-3P"
+		(property "Footprint" "Custom SamacSys Footprints:TO130P160X410X300-3P"
 			(at 352.73 33.02 0)
 			(effects
@@
 			)
 		)
-		(property "Footprint" "TO130P160X410X300-3P"
+		(property "Footprint" "Custom SamacSys Footprints:TO130P160X410X300-3P"
 			(at 167.97 119.38 0)
 			(effects
@@
 			)
 		)
-		(property "Footprint" "TO130P160X410X300-3P"
+		(property "Footprint" "Custom SamacSys Footprints:TO130P160X410X300-3P"
 			(at 238.43 33.02 0)
 			(effects
@@
 			)
 		)
-		(property "Footprint" "TO130P160X410X300-3P"
+		(property "Footprint" "Custom SamacSys Footprints:TO130P160X410X300-3P"
 			(at 34.62 119.38 0)
 			(effects
@@
 			)
 		)
-		(property "Footprint" "TO130P160X410X300-3P"
+		(property "Footprint" "Custom SamacSys Footprints:TO130P160X410X300-3P"
 			(at 276.53 33.02 0)
 			(effects
@@
 			)
 		)
-		(property "Footprint" "TO130P160X410X300-3P"
+		(property "Footprint" "Custom SamacSys Footprints:TO130P160X410X300-3P"
 			(at 91.77 119.38 0)
 			(effects
@@
 			)
 		)
-		(property "Footprint" "TO130P160X410X300-3P"
+		(property "Footprint" "Custom SamacSys Footprints:TO130P160X410X300-3P"
 			(at 129.87 119.38 0)
 			(effects
@@
 			)
 		)
-		(property "Footprint" "TO130P160X410X300-3P"
+		(property "Footprint" "Custom SamacSys Footprints:TO130P160X410X300-3P"
 			(at 333.68 33.02 0)
 			(effects
@@
 	)
 	(symbol
+		(lib_name "SS49E_1")
 		(lib_id "Custom SamacSys Symbols:SS49E")
 		(at 124.46 49.53 90)
@@
 			)
 		)
-		(property "Footprint" "TO130P160X410X300-3P"
+		(property "Footprint" "Custom SamacSys Footprints:TO130P160X410X300-3P"
 			(at 219.38 33.02 0)
 			(effects

Commit message: Widen power traces
Parts:
- IC1, IC10, IC11, IC12, IC13, IC14, IC15, IC16, IC2, IC3, IC4, IC5, IC6, IC7, IC8, IC9: DigiKey Price/Stock (none) -> https://www.digikey.com/short/592nmtp5
- U1: DigiKey Price/Stock (none) -> https://www.digikey.com/short/0jjmqb9w
Changed lines of the file:
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@@
 			)
 		)
+		(property "DigiKey Price/Stock" "https://www.digikey.com/short/592nmtp5"
+			(at 205.74 102.87 0)
+			(effects
+				(font
+					(size 1.27 1.27)
+				)
+				(hide yes)
+			)
+		)
 		(pin "1"
 		)
@@
 			)
 		)
+		(property "DigiKey Price/Stock" "https://www.digikey.com/short/592nmtp5"
+			(at 162.56 49.53 0)
+			(effects
+				(font
+					(size 1.27 1.27)
+				)
+				(hide yes)
+			)
+		)
 		(pin "1"
 		)
@@
 			)
 		)
+		(property "DigiKey Price/Stock" "https://www.digikey.com/short/0jjmqb9w"
+			(at 85.09 74.93 0)
+			(effects
+				(font
+					(size 1.27 1.27)
+				)
+				(hide yes)
+			)
+		)
 		(pin "22"
 		)
@@
 			)
 		)
+		(property "DigiKey Price/Stock" "https://www.digikey.com/short/592nmtp5"
+			(at 167.64 102.87 0)
+			(effects
+				(font
+					(size 1.27 1.27)
+				)
+				(hide yes)
+			)
+		)
 		(pin "1"
 		)
@@
 			)
 		)
+		(property "DigiKey Price/Stock" "https://www.digikey.com/short/592nmtp5"
+			(at 243.84 102.87 0)
+			(effects
+				(font
+					(size 1.27 1.27)
+				)
+				(hide yes)
+			)
+		)
 		(pin "1"
 		)
@@
 			)
 		)
+		(property "DigiKey Price/Stock" "https://www.digikey.com/short/592nmtp5"
+			(at 148.59 102.87 0)
+			(effects
+				(font
+					(size 1.27 1.27)
+				)
+				(hide yes)
+			)
+		)
 		(pin "1"
 		)
@@
 			)
 		)
+		(property "DigiKey Price/Stock" ""
+			(at 41.91 69.85 0)
+			(effects
+				(font
+					(size 1.27 1.27)
+				)
+				(hide yes)
+			)
+		)
 		(pin "8"
 		)
@@
 			)
 		)
+		(property "DigiKey Price/Stock" "https://www.digikey.com/short/592nmtp5"
+			(at 219.71 49.53 0)
+			(effects
+				(font
+					(size 1.27 1.27)
+				)
+				(hide yes)
+			)
+		)
 		(pin "1"
 		)
@@
 			)
 		)
+		(property "DigiKey Price/Stock" "https://www.digikey.com/short/592nmtp5"
+			(at 200.66 49.53 0)
+			(effects
+				(font
+					(size 1.27 1.27)
+				)
+				(hide yes)
+			)
+		)
 		(pin "1"
 		)
@@
 			)
 		)
+		(property "DigiKey Price/Stock" "https://www.digikey.com/short/592nmtp5"
+			(at 257.81 49.53 0)
+			(effects
+				(font
+					(size 1.27 1.27)
+				)
+				(hide yes)
+			)
+		)
 		(pin "1"
 		)
@@
 			)
 		)
+		(property "DigiKey Price/Stock" "https://www.digikey.com/short/592nmtp5"
+			(at 262.89 102.87 0)
+			(effects
+				(font
+					(size 1.27 1.27)
+				)
+				(hide yes)
+			)
+		)
 		(pin "1"
 		)
@@
 			)
 		)
+		(property "DigiKey Price/Stock" "https://www.digikey.com/short/592nmtp5"
+			(at 143.51 49.53 0)
+			(effects
+				(font
+					(size 1.27 1.27)
+				)
+				(hide yes)
+			)
+		)
 		(pin "1"
 		)
@@
 			)
 		)
+		(property "DigiKey Price/Stock" "https://www.digikey.com/short/592nmtp5"
+			(at 129.54 102.87 0)
+			(effects
+				(font
+					(size 1.27 1.27)
+				)
+				(hide yes)
+			)
+		)
 		(pin "1"
 		)
@@
 			)
 		)
+		(property "DigiKey Price/Stock" ""
+			(at 78.74 46.99 0)
+			(effects
+				(font
+					(size 1.27 1.27)
+				)
+				(hide yes)
+			)
+		)
 		(pin "1"
 		)
@@
 			)
 		)
+		(property "DigiKey Price/Stock" "https://www.digikey.com/short/592nmtp5"
+			(at 181.61 49.53 0)
+			(effects
+				(font
+					(size 1.27 1.27)
+				)
+				(hide yes)
+			)
+		)
 		(pin "1"
 		)
@@
 			)
 		)
+		(property "DigiKey Price/Stock" "https://www.digikey.com/short/592nmtp5"
+			(at 186.69 102.87 0)
+			(effects
+				(font
+					(size 1.27 1.27)
+				)
+				(hide yes)
+			)
+		)
 		(pin "1"
 		)
@@
 			)
 		)
+		(property "DigiKey Price/Stock" "https://www.digikey.com/short/592nmtp5"
+			(at 224.79 102.87 0)
+			(effects
+				(font
+					(size 1.27 1.27)
+				)
+				(hide yes)
+			)
+		)
 		(pin "1"
 		)
@@
 			)
 		)
+		(property "DigiKey Price/Stock" "https://www.digikey.com/short/592nmtp5"
+			(at 238.76 49.53 0)
+			(effects
+				(font
+					(size 1.27 1.27)
+				)
+				(hide yes)
+			)
+		)
 		(pin "1"
 		)
@@
 				(hide yes)
 			)
+		)
+		(property "DigiKey Price/Stock" "https://www.digikey.com/short/592nmtp5"
+			(at 124.46 49.53 0)
+			(effects
+				(font
+					(size 1.27 1.27)
+				)
+				(hide yes)
+			)
