File: Chessboard Hardware.kicad_sch (KiCad schematic)
At the start: 15 parts, among them J1 Conn_01x04_Pin

Commit message: Done
Parts:
- added H1, H2, H3, H4: MountingHole, MountingHole:MountingHole_2.7mm_M2.5, symbol Mechanical:MountingHole
