File: Chessboard Eighth.kicad_sch (KiCad schematic)
At the start: 9 parts

Commit message: Reannoate
Parts:
- renumbered U11 to U20, U3 to U21, U4 to U22, U5 to U23, U15 to U24, U7 to U25, U8 to U26, U9 to U27, U10 to U28

Commit message: Simpler schematic with one less chip, use UART for comms
Parts:
- renumbered U20 to U19, U21 to U20, U22 to U21, U23 to U22, U24 to U23, U25 to U24, U26 to U25, U27 to U26, U28 to U27

Commit message: Oops forgot decoupling caps
Parts:
- added C3: 100nF, Capacitor_THT:C_Disc_D5.0mm_W2.5mm_P2.50mm, symbol Device:C
Connections:
- net GND: now also C3.1
- net VCC: now also C3.2
Changed lines of the file:
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@@
 	(generator_version "8.0")
 	(paper "A4")
+	(junction
+		(at 66.04 44.45)
+		(diameter 0)
+		(color 0 0 0 0)
+	)
 	(wire
 		(pts
@@
 	(wire
 		(pts
-			(xy 78.74 55.88) (xy 104.14 55.88)
+			(xy 66.04 41.91) (xy 66.04 44.45)
 		)
 		(stroke
@@
 	(wire
 		(pts
-			(xy 104.14 73.66) (xy 104.14 93.98)
+			(xy 78.74 55.88) (xy 104.14 55.88)
 		)
 		(stroke
@@
 	(wire
 		(pts
-			(xy 144.78 35.56) (xy 144.78 60.96)
+			(xy 104.14 73.66) (xy 104.14 93.98)
 		)
 		(stroke
@@
 	(wire
 		(pts
-			(xy 124.46 71.12) (xy 124.46 93.98)
+			(xy 144.78 35.56) (xy 144.78 60.96)
 		)
 		(stroke
@@
 	(wire
 		(pts
-			(xy 78.74 63.5) (xy 165.1 63.5)
+			(xy 124.46 71.12) (xy 124.46 93.98)
 		)
 		(stroke
@@
 	(wire
 		(pts
-			(xy 104.14 55.88) (xy 104.14 35.56)
+			(xy 78.74 63.5) (xy 165.1 63.5)
 		)
 		(stroke
@@
 	(wire
 		(pts
+			(xy 104.14 55.88) (xy 104.14 35.56)
+		)
+		(stroke
+			(width 0)
+			(type default)
+		)
+	)
+	(wire
+		(pts
 			(xy 144.78 68.58) (xy 144.78 93.98)
+		)
+		(stroke
+			(width 0)
+			(type default)
+		)
+	)
+	(wire
+		(pts
+			(xy 66.04 44.45) (xy 66.04 49.53)
 		)
 		(stroke
@@
 	(symbol
 		(lib_id "power:VCC")
-		(at 66.04 49.53 0)
+		(at 66.04 41.91 0)
 		(unit 1)
 		(exclude_from_sim no)
@@
 		(fields_autoplaced yes)
 		(property "Reference" "#PWR052"
-			(at 66.04 53.34 0)
+			(at 66.04 45.72 0)
 			(effects
 				(font
@@
 		)
 		(property "Value" "VCC"
-			(at 66.04 44.45 0)
+			(at 66.04 36.83 0)
 			(effects
 				(font
@@
 		)
 		(property "Footprint" ""
-			(at 66.04 49.53 0)
+			(at 66.04 41.91 0)
 			(effects
 				(font
@@
 		)
 		(property "Datasheet" ""
-			(at 66.04 49.53 0)
+			(at 66.04 41.91 0)
 			(effects
 				(font
@@
 		)
 		(property "Description" "Power symbol creates a global label with name \"VCC\""
-			(at 66.04 49.53 0)
+			(at 66.04 41.91 0)
 			(effects
 				(font
@@
 	)
 	(symbol
+		(lib_id "Device:C")
+		(at 62.23 44.45 90)
+		(unit 1)
+		(exclude_from_sim no)
+		(in_bom yes)
+		(on_board yes)
+		(dnp no)
+		(fields_autoplaced yes)
+		(property "Reference" "C3"
+			(at 62.23 36.83 90)
+			(effects
+				(font
+					(size 1.27 1.27)
+				)
+			)
+		)
+		(property "Value" "100nF"
+			(at 62.23 39.37 90)
+			(effects
+				(font
+					(size 1.27 1.27)
+				)
+			)
+		)
+		(property "Footprint" "Capacitor_THT:C_Disc_D5.0mm_W2.5mm_P2.50mm"
+			(at 66.04 43.4848 0)
+			(effects
+				(font
+					(size 1.27 1.27)
+				)
+				(hide yes)
+			)
+		)
+		(property "Datasheet" "~"
+			(at 62.23 44.45 0)
+			(effects
+				(font
+					(size 1.27 1.27)
+				)
+				(hide yes)
+			)
+		)
+		(property "Description" "Unpolarized capacitor"
+			(at 62.23 44.45 0)
+			(effects
+				(font
+					(size 1.27 1.27)
+				)
+				(hide yes)
+			)
+		)
+		(pin "2"
+		)
+		(pin "1"
+		)
+		(instances
+			(project ""
+				(path "/e63e39d7-6ac0-4ffd-8aa3-1841a4541b55/0a97662c-6566-4e1d-afc5-82a5fb54d5c1"
+					(reference "C3")
+					(unit 1)
+				)
+				(path "/e63e39d7-6ac0-4ffd-8aa3-1841a4541b55/2cc389a0-19b7-477f-9935-260f74c2b165"
+					(reference "C5")
+					(unit 1)
+				)
+				(path "/e63e39d7-6ac0-4ffd-8aa3-1841a4541b55/5515513e-868f-4ac2-8212-63f927d4c305"
+					(reference "C4")
+					(unit 1)
+				)
+				(path "/e63e39d7-6ac0-4ffd-8aa3-1841a4541b55/6ff0f717-87ae-4710-96ea-9ed2085024e0"
+					(reference "C8")
+					(unit 1)
+				)
+				(path "/e63e39d7-6ac0-4ffd-8aa3-1841a4541b55/7201e36b-84cd-4f5e-823d-16da688e57ec"
+					(reference "C2")
+					(unit 1)
+				)
+				(path "/e63e39d7-6ac0-4ffd-8aa3-1841a4541b55/9ab27e34-a744-41d7-b2b4-f273a8bfac2f"
+					(reference "C7")
+					(unit 1)
+				)
+				(path "/e63e39d7-6ac0-4ffd-8aa3-1841a4541b55/b56c74a5-7b5e-4776-9f0a-48333d5f8270"
+					(reference "C1")
+					(unit 1)
+				)
+				(path "/e63e39d7-6ac0-4ffd-8aa3-1841a4541b55/e9fb6c6b-71dd-42a0-a36e-8962cbc1247e"
+					(reference "C6")
+					(unit 1)
+				)
+			)
+		)
+	)
+	(symbol
 		(lib_id "power:VCC")
 		(at 156.21 82.55 0)
@@
 					(unit 1)
 				)
+			)
+		)
+	)
+	(symbol
+		(lib_id "power:GND")
+		(at 58.42 44.45 0)
+		(unit 1)
+		(exclude_from_sim no)
+		(in_bom yes)
+		(on_board yes)
+		(dnp no)
+		(fields_autoplaced yes)
+		(property "Reference" "#PWR0154"
+			(at 58.42 50.8 0)
+			(effects
+				(font
+					(size 1.27 1.27)
+				)
+				(hide yes)
+			)
+		)
+		(property "Value" "GND"
+			(at 58.42 49.53 0)
+			(effects
+				(font
+					(size 1.27 1.27)
+				)
+			)
+		)
+		(property "Footprint" ""
+			(at 58.42 44.45 0)
+			(effects
+				(font
+					(size 1.27 1.27)
+				)
+				(hide yes)
+			)
+		)
+		(property "Datasheet" ""
+			(at 58.42 44.45 0)
+			(effects
+				(font
+					(size 1.27 1.27)
+				)
+				(hide yes)
+			)
+		)
+		(property "Description" "Power symbol creates a global label with name \"GND\" , ground"
+			(at 58.42 44.45 0)
+			(effects
+				(font
+					(size 1.27 1.27)
+				)
+				(hide yes)
+			)
+		)
+		(pin "1"
+		)
+		(instances
+			(project ""
+				(path "/e63e39d7-6ac0-4ffd-8aa3-1841a4541b55/0a97662c-6566-4e1d-afc5-82a5fb54d5c1"
+					(reference "#PWR0154")
+					(unit 1)
+				)
+				(path "/e63e39d7-6ac0-4ffd-8aa3-1841a4541b55/2cc389a0-19b7-477f-9935-260f74c2b165"
+					(reference "#PWR0156")
+					(unit 1)
+				)
+				(path "/e63e39d7-6ac0-4ffd-8aa3-1841a4541b55/5515513e-868f-4ac2-8212-63f927d4c305"
+					(reference "#PWR0155")
+					(unit 1)
+				)
+				(path "/e63e39d7-6ac0-4ffd-8aa3-1841a4541b55/6ff0f717-87ae-4710-96ea-9ed2085024e0"
+					(reference "#PWR0159")
+					(unit 1)
+				)
+				(path "/e63e39d7-6ac0-4ffd-8aa3-1841a4541b55/7201e36b-84cd-4f5e-823d-16da688e57ec"
+					(reference "#PWR0153")
+					(unit 1)
+				)
+				(path "/e63e39d7-6ac0-4ffd-8aa3-1841a4541b55/9ab27e34-a744-41d7-b2b4-f273a8bfac2f"
+					(reference "#PWR0158")
+					(unit 1)
+				)
+				(path "/e63e39d7-6ac0-4ffd-8aa3-1841a4541b55/b56c74a5-7b5e-4776-9f0a-48333d5f8270"
+					(reference "#PWR0152")
+					(unit 1)
+				)
+				(path "/e63e39d7-6ac0-4ffd-8aa3-1841a4541b55/e9fb6c6b-71dd-42a0-a36e-8962cbc1247e"
+					(reference "#PWR0157")
+					(unit 1)
+				)
