File: Sensor Quarter/Sensor Quarter.kicad_pcb (KiCad board)
At the start: 2 copper layers, 100 x 100 mm, 19 parts, among them IC1 SS49E, IC10 SS49E, IC11 SS49E, IC12 SS49E, IC13 SS49E, IC14 SS49E, IC15 SS49E, IC16 SS49E, IC2 SS49E, IC3 SS49E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

Commit message: Again
Parts:
- added J2: Conn_01x02_Pin, Connector_PinHeader_2.54mm:PinHeader_1x02_P2.54mm_Vertical, F.Cu at (51.8, 51.8)
- added J3: Conn_01x02_Pin, Connector_PinHeader_2.54mm:PinHeader_1x02_P2.54mm_Vertical, F.Cu at (51.8, 145.7)
- added J4: Conn_01x02_Pin, Connector_PinHeader_2.54mm:PinHeader_1x02_P2.54mm_Vertical, F.Cu at (148.2, 145.7)
- moved C1 5.00 mm to (112.0, 102.6)
- moved U1 0.15 mm to (99.8, 99.8)
Routing:
- net GND: track 422.8 -> 618.5 mm, vias 2 -> 4
- net VCC: track 437.1 -> 618.4 mm, vias 3 -> 4
- net Net-(IC13-O): track 53.5 -> 63.0 mm, vias 1 -> 0
- net Net-(J1-Pin_3): track 82.4 -> 74.8 mm
- net Net-(J1-Pin_7): track 79.0 -> 71.6 mm, vias 0 -> 1
- net Net-(IC11-O): track 24.2 -> 18.4 mm
- net Net-(J1-Pin_8): track 70.0 -> 74.4 mm
- net Net-(IC16-O): track 63.0 -> 67.0 mm
- net Net-(IC4-O): track 51.5 -> 55.3 mm
- net Net-(J1-Pin_5): track 71.7 -> 69.0 mm, vias 2 -> 1
- net Net-(IC5-O): track 41.1 -> 43.3 mm, vias 0 -> 1
- net Net-(IC10-O): track 24.3 -> 22.9 mm, vias 0 -> 1
- net Net-(IC9-O): track 50.9 -> 49.8 mm, vias 0 -> 1
- net Net-(IC6-O): track 17.7 -> 17.0 mm
- net Net-(J1-Pin_6): track 70.4 -> 69.9 mm, vias 2 -> 1
Other:
- board text removed: "Linear hall 4x4 grid with CD74HC4067M for chessboard"
- board text removed: "VCC GND SIG Flat side down"
