File: Sensor Quarter/Sensor Quarter.kicad_sch (KiCad schematic)
At the start: 19 parts, among them IC1 SS49E, IC10 SS49E, IC11 SS49E, IC12 SS49E, IC13 SS49E, IC14 SS49E, IC15 SS49E, IC16 SS49E, IC2 SS49E, IC3 SS49E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

Commit message: Move to own directory because we'll have multiple KiCad projects
Other:
- title: Chessboard Hardware - Chessboard sensor quarter -> Chessboard Hardware - Sensor quarter
Changed lines of the file:
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@@
 	(paper "A4")
 	(title_block
-		(title "Chessboard Hardware - Chessboard sensor quarter")
+		(title "Chessboard Hardware - Sensor quarter")
 		(rev "0")
 		(comment 1 "This is only one quarter of the entire sensing array.")

Commit message: Again
Parts:
- added J2, J3, J4: Conn_01x02_Pin, Connector_PinHeader_2.54mm:PinHeader_1x02_P2.54mm_Vertical, symbol Connector:Conn_01x02_Pin
Connections:
- net GND: now also J2.2 (Pin_2), J3.2 (Pin_2), J4.2 (Pin_2)
- net VCC: now also J2.1 (Pin_1), J3.1 (Pin_1), J4.1 (Pin_1)
